File: Timer.kicad_pcb (KiCad board)
At the start: 2 copper layers, 110 x 62.5 mm, 36 parts, among them IC1 ATTINY85-P, P1 LEDS, P2 PWR, Q1 BC547, Q2 BC547, SW1 START/STOP, SW2 +M, SW3 -M, SW4 +S, SW5 -S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

Commit message: Updated PCB
Routing:
- net Net-(DS1-Pad5): track 52.5 -> 27.6 mm
Changed lines of the file:
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@@
   (general
     (links 78)
-    (no_connects 10)
+    (no_connects 0)
     (area 137.424999 64.924999 247.575001 127.575001)
     (thickness 1.6)
     (drawings 4)
-    (tracks 308)
+    (tracks 295)
     (zones 0)
     (modules 36)
@@
   (gr_line (start 137.5 127.5) (end 247.5 127.5) (layer Edge.Cuts) (width 0.15))
   (gr_line (start 137.5 65) (end 137.5 127.5) (layer Edge.Cuts) (width 0.15))
-  (segment (start 241.3 97.635) (end 230.223 97.635) (width 1.8) (layer B.Cu) (net 1))
-  (segment (start 227.457 94.869) (end 227.457 90.326841) (width 1.8) (layer B.Cu) (net 1))
-  (segment (start 230.223 97.635) (end 227.457 94.869) (width 1.8) (layer B.Cu) (net 1))
-  (segment (start 227.457 90.326841) (end 227.469001 90.31484) (width 1.8) (layer B.Cu) (net 1))
-  (segment (start 238.76 75.473781) (end 238.76 72.644) (width 1.8) (layer B.Cu) (net 1))
-  (segment (start 238.76 72.644) (end 238.887 72.517) (width 1.8) (layer B.Cu) (net 1))
-  (segment (start 227.469001 90.31484) (end 227.469001 86.76478) (width 1.8) (layer B.Cu) (net 1))
-  (segment (start 227.469001 86.76478) (end 238.76 75.473781) (width 1.8) (layer B.Cu) (net 1))
+  (segment (start 241.3 97.635) (end 230.223 97.635) (width 1) (layer B.Cu) (net 1))
+  (segment (start 227.457 94.869) (end 227.457 90.326841) (width 1) (layer B.Cu) (net 1))
+  (segment (start 230.223 97.635) (end 227.457 94.869) (width 1) (layer B.Cu) (net 1))
+  (segment (start 227.457 90.326841) (end 227.469001 90.31484) (width 1) (layer B.Cu) (net 1))
+  (segment (start 238.76 75.473781) (end 238.76 72.644) (width 1) (layer B.Cu) (net 1))
+  (segment (start 238.76 72.644) (end 238.887 72.517) (width 1) (layer B.Cu) (net 1))
+  (segment (start 227.469001 90.31484) (end 227.469001 86.76478) (width 1) (layer B.Cu) (net 1))
+  (segment (start 227.469001 86.76478) (end 238.76 75.473781) (width 1) (layer B.Cu) (net 1))
   (segment (start 155.53436 89.57564) (end 156.771839 89.57564) (width 1) (layer B.Cu) (net 2))
   (segment (start 187.452 85.344) (end 187.452 82.48218) (width 1) (layer B.Cu) (net 2))
@@
   (segment (start 148.59 78.58557) (end 154.45943 84.455) (width 1) (layer B.Cu) (net 2))
   (segment (start 154.45943 84.455) (end 156.21 84.455) (width 1) (layer B.Cu) (net 2))
-  (segment (start 241.3 82.705) (end 234.922 82.705) (width 1.8) (layer B.Cu) (net 2))
-  (segment (start 234.922 82.705) (end 230.009001 87.617999) (width 1.8) (layer B.Cu) (net 2))
-  (segment (start 230.009001 87.617999) (end 230.009001 90.31484) (width 1.8) (layer B.Cu) (net 2))
-  (segment (start 230.009001 90.31484) (end 230.009001 93.992001) (width 1.8) (layer B.Cu) (net 2))
-  (segment (start 230.009001 93.992001) (end 231.14 95.123) (width 1.8) (layer B.Cu) (net 2))
-  (segment (start 231.14 95.123) (end 239.039208 95.123) (width 1.8) (layer B.Cu) (net 2))
-  (segment (start 239.039208 95.123) (end 240.027208 94.135) (width 1.8) (layer B.Cu) (net 2))
-  (segment (start 240.027208 94.135) (end 241.3 94.135) (width 1.8) (layer B.Cu) (net 2))
-  (segment (start 243.967 72.517) (end 243.967 80.038) (width 1.8) (layer B.Cu) (net 2))
-  (segment (start 243.967 80.038) (end 241.3 82.705) (width 1.8) (layer B.Cu) (net 2))
+  (segment (start 241.3 82.705) (end 234.922 82.705) (width 1) (layer B.Cu) (net 2))
+  (segment (start 234.922 82.705) (end 230.009001 87.617999) (width 1) (layer B.Cu) (net 2))
+  (segment (start 230.009001 87.617999) (end 230.009001 90.31484) (width 1) (layer B.Cu) (net 2))
+  (segment (start 230.009001 90.31484) (end 230.009001 93.992001) (width 1) (layer B.Cu) (net 2))
+  (segment (start 230.009001 93.992001) (end 231.14 95.123) (width 1) (layer B.Cu) (net 2))
+  (segment (start 231.14 95.123) (end 239.039208 95.123) (width 1) (layer B.Cu) (net 2))
+  (segment (start 239.039208 95.123) (end 240.027208 94.135) (width 1) (layer B.Cu) (net 2))
+  (segment (start 240.027208 94.135) (end 241.3 94.135) (width 1) (layer B.Cu) (net 2))
+  (segment (start 243.967 72.517) (end 243.967 80.038) (width 1) (layer B.Cu) (net 2))
+  (segment (start 243.967 80.038) (end 241.3 82.705) (width 1) (layer B.Cu) (net 2))
   (segment (start 156.21 76.835) (end 156.21 75.438) (width 0.4) (layer B.Cu) (net 3))
   (segment (start 162.56 73.152) (end 162.56 67.93399) (width 0.4) (layer B.Cu) (net 3))
@@
   (segment (start 150.55199 67.80699) (end 151.13 68.385) (width 1) (layer B.Cu) (net 3))
   (segment (start 151.13 68.385) (end 151.13 70.485) (width 1) (layer B.Cu) (net 3))
-  (segment (start 241.3 86.205) (end 241.3 88.138) (width 1.8) (layer B.Cu) (net 3))
-  (segment (start 241.3 88.138) (end 244.348 91.186) (width 1.8) (layer B.Cu) (net 3))
-  (segment (start 244.348 91.186) (end 244.348 100.838) (width 1.8) (layer B.Cu) (net 3))
-  (segment (start 244.348 100.838) (end 242.686 102.5) (width 1.8) (layer B.Cu) (net 3))
-  (segment (start 242.686 102.5) (end 224.74 102.5) (width 1.8) (layer B.Cu) (net 3))
-  (segment (start 224.74 102.5) (end 219.404999 107.835001) (width 1.8) (layer B.Cu) (net 3))
-  (segment (start 219.404999 107.835001) (end 218.305 108.935) (width 1.8) (layer B.Cu) (net 3))
+  (segment (start 241.3 86.205) (end 241.3 88.138) (width 1) (layer B.Cu) (net 3))
+  (segment (start 241.3 88.138) (end 244.348 91.186) (width 1) (layer B.Cu) (net 3))
+  (segment (start 244.348 91.186) (end 244.348 100.838) (width 1) (layer B.Cu) (net 3))
+  (segment (start 244.348 100.838) (end 242.686 102.5) (width 1) (layer B.Cu) (net 3))
+  (segment (start 242.686 102.5) (end 224.74 102.5) (width 1) (layer B.Cu) (net 3))
+  (segment (start 224.74 102.5) (end 219.404999 107.835001) (width 1) (layer B.Cu) (net 3))
+  (segment (start 219.404999 107.835001) (end 218.305 108.935) (width 1) (layer B.Cu) (net 3))
   (segment (start 212.09 111.125) (end 216.115 111.125) (width 1) (layer B.Cu) (net 3))
   (segment (start 216.115 111.125) (end 218.305 108.935) (width 1) (layer B.Cu) (net 3))
   (segment (start 177.45456 107.8738) (end 180.70576 111.125) (width 1) (layer B.Cu) (net 3))
   (segment (start 180.70576 111.125) (end 212.09 111.125) (width 1) (layer B.Cu) (net 3))
-  (segment (start 232.549001 90.31484) (end 237.19016 90.31484) (width 1.8) (layer B.Cu) (net 3))
-  (segment (start 237.19016 90.31484) (end 241.3 86.205) (width 1.8) (layer B.Cu) (net 3))
+  (segment (start 232.549001 90.31484) (end 237.19016 90.31484) (width 1) (layer B.Cu) (net 3))
+  (segment (start 237.19016 90.31484) (end 241.3 86.205) (width 1) (layer B.Cu) (net 3))
   (segment (start 151.13 70.485) (end 151.13 69.763458) (width 0.4) (layer B.Cu) (net 3))
   (segment (start 212.09 118.745) (end 212.09 120.65) (width 1) (layer B.Cu) (net 4))
@@
   (segment (start 153.162 75.438) (end 156.21 72.39) (width 0.4) (layer B.Cu) (net 6))
   (segment (start 156.21 72.39) (end 156.21 70.485) (width 0.4) (layer B.Cu) (net 6))
-  (segment (start 170.18 88.828585) (end 170.18 91.44) (width 0.4) (layer B.Cu) (net 7))
-  (segment (start 170.18 91.44) (end 170.84999 92.10999) (width 0.4) (layer B.Cu) (net 7))
-  (segment (start 170.84999 92.10999) (end 172.08077 92.10999) (width 0.4) (layer B.Cu) (net 7))
-  (segment (start 172.08077 92.10999) (end 172.72 91.47076) (width 0.4) (layer B.Cu) (net 7))
-  (segment (start 172.72 91.47076) (end 172.72 83.532587) (width 0.4) (layer B.Cu) (net 7))
-  (segment (start 172.72 83.532587) (end 172.142583 82.95517) (width 0.4) (layer B.Cu) (net 7))
-  (segment (start 172.142583 82.95517) (end 170.734575 82.95517) (width 0.4) (layer B.Cu) (net 7))
-  (segment (start 170.734575 82.95517) (end 170.18 83.509745) (width 0.4) (layer B.Cu) (net 7))
-  (segment (start 170.18 83.509745) (end 170.18 85.979) (width 0.4) (layer B.Cu) (net 7))
-  (segment (start 170.18 85.979) (end 169.672 86.487) (width 0.4) (layer B.Cu) (net 7))
-  (segment (start 166.37 85.979) (end 166.37 84.455) (width 0.4) (layer B.Cu) (net 7))
-  (segment (start 169.672 86.487) (end 166.878 86.487) (width 0.4) (layer B.Cu) (net 7))
-  (segment (start 166.878 86.487) (end 166.37 85.979) (width 0.4) (layer B.Cu) (net 7))
   (segment (start 157.093529 81.949987) (end 157.09353 81.949989) (width 0.4) (layer B.Cu) (net 7))
   (segment (start 157.09353 81.949989) (end 165.515989 81.949989) (width 0.4) (layer B.Cu) (net 7))
@@
   (segment (start 193.779967 80.540033) (end 194.945 79.375) (width 0.4) (layer B.Cu) (net 23))
   (segment (start 194.945 79.375) (end 194.945 76.835) (width 0.4) (layer B.Cu) (net 23))
-  (segment (start 241.3 112.395) (end 218.845 112.395) (width 1.8) (layer B.Cu) (net 24))
-  (segment (start 218.845 112.395) (end 216.305 114.935) (width 1.8) (layer B.Cu) (net 24))
-  (segment (start 233.965 117.475) (end 241.3 117.475) (width 1.8) (layer B.Cu) (net 25))
-  (segment (start 230.505 120.935) (end 233.965 117.475) (width 1.8) (layer B.Cu) (net 25))
+  (segment (start 241.3 112.395) (end 218.845 112.395) (width 1) (layer B.Cu) (net 24))
+  (segment (start 218.845 112.395) (end 216.305 114.935) (width 1) (layer B.Cu) (net 24))
+  (segment (start 233.965 117.475) (end 241.3 117.475) (width 1) (layer B.Cu) (net 25))
+  (segment (start 230.505 120.935) (end 233.965 117.475) (width 1) (layer B.Cu) (net 25))
   (segment (start 209.041999 121.158001) (end 208.28 121.92) (width 0.4) (layer B.Cu) (net 26))
   (segment (start 210.439 114.937806) (end 210.439 119.761) (width 0.4) (layer B.Cu) (net 26))

Commit message: Some Photos Added
Other:
- board text added: "+ -"
Changed lines of the file:
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@@
     (area 137.424999 64.924999 247.575001 127.575001)
     (thickness 1.6)
-    (drawings 4)
+    (drawings 5)
     (tracks 295)
     (zones 0)
@@
     )
   )
+  (gr_text "+   -" (at 241.3 66.294) (layer F.SilkS)
+    (effects (font (size 1.8 1.8) (thickness 0.4)))
+  )
   (gr_line (start 247.5 65) (end 137.5 65) (layer Edge.Cuts) (width 0.15))
